File: plank.kicad_pcb (KiCad board)
At the start: 2 copper layers, 212 parts, among them SW1 SW_Push, U1 ATmega32U4-A, Y1 16MHz

Commit message: Switches in place
Parts:
- moved MX88 257.4 mm to (391.5, 33.0)
- moved D76 242.1 mm to (495.3, 45.1)
- moved D77 242.1 mm to (495.3, 48.4)
- moved D78 242.1 mm to (495.3, 51.8)
- moved D79 242.1 mm to (495.3, 55.1)
- moved D80 242.1 mm to (495.3, 58.5)
- moved D81 242.1 mm to (495.3, 61.8)
- moved D82 242.1 mm to (495.3, 65.2)
- moved D83 242.1 mm to (495.3, 68.5)
- moved D84 242.1 mm to (495.3, 71.9)
- moved D85 242.1 mm to (495.3, 75.2)
- moved D86 242.1 mm to (495.3, 78.6)
- moved D87 242.1 mm to (495.3, 81.9)
- moved D88 242.1 mm to (495.3, 85.3)
- moved D89 242.1 mm to (495.3, 88.6)
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
Commit message: Added edge and bolt locations
Other:
- board outline added: 420.7 x 164.3 mm
Changed lines of the file:
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@@
     )
   )
+  (gr_circle (center 169.06875 149.225) (end 173.83125 149.225)
+    (stroke (width 0.1) (type default)) (fill none) (layer "Edge.Cuts"))
+  (gr_circle (center 51.59375 -5.55625) (end 56.35625 -5.55625)
+    (stroke (width 0.1) (type default)) (fill none) (layer "Edge.Cuts"))
+  (gr_circle (center 110.33125 149.225) (end 115.09375 149.225)
+    (stroke (width 0.1) (type default)) (fill none) (layer "Edge.Cuts"))
+  (gr_line (start -7.14375 -10.31875) (end 403.225 -10.31875)
+    (stroke (width 0.1) (type default)) (layer "Edge.Cuts"))
+  (gr_circle (center -7.14375 -5.55625) (end -2.38125 -5.55625)
+    (stroke (width 0.1) (type default)) (fill none) (layer "Edge.Cuts"))
+  (gr_circle (center 404.01875 46.0375) (end 404.01875 41.275)
+    (stroke (width 0.1) (type default)) (fill none) (layer "Edge.Cuts"))
+  (gr_line (start -11.90625 149.225) (end -11.90625 -5.55625)
+    (stroke (width 0.1) (type default)) (layer "Edge.Cuts"))
+  (gr_circle (center 404.01875 149.225) (end 404.01875 144.4625)
+    (stroke (width 0.1) (type default)) (fill none) (layer "Edge.Cuts"))
+  (gr_circle (center -7.14375 149.225) (end -2.38125 149.225)
+    (stroke (width 0.1) (type default)) (fill none) (layer "Edge.Cuts"))
+  (gr_circle (center 51.59375 149.225) (end 56.35625 149.225)
+    (stroke (width 0.1) (type default)) (fill none) (layer "Edge.Cuts"))
+  (gr_circle (center 286.54375 149.225) (end 291.30625 149.225)
+    (stroke (width 0.1) (type default)) (fill none) (layer "Edge.Cuts"))
+  (gr_circle (center 404.01875 97.63125) (end 404.01875 92.86875)
+    (stroke (width 0.1) (type default)) (fill none) (layer "Edge.Cuts"))
+  (gr_line (start 408.78125 -6.35) (end 408.78125 149.225)
+    (stroke (width 0.1) (type default)) (layer "Edge.Cuts"))
+  (gr_line (start 404.01875 153.9875) (end -7.14375 153.9875)
+    (stroke (width 0.1) (type default)) (layer "Edge.Cuts"))
+  (gr_circle (center 345.28125 149.225) (end 350.04375 149.225)
+    (stroke (width 0.1) (type default)) (fill none) (layer "Edge.Cuts"))
+  (gr_circle (center 169.06875 -5.55625) (end 173.83125 -5.55625)
+    (stroke (width 0.1) (type default)) (fill none) (layer "Edge.Cuts"))
+  (gr_circle (center 227.80625 149.225) (end 232.56875 149.225)
+    (stroke (width 0.1) (type default)) (fill none) (layer "Edge.Cuts"))
+  (gr_circle (center -7.14375 97.63125) (end -7.14375 92.86875)
+    (stroke (width 0.1) (type default)) (fill none) (layer "Edge.Cuts"))
+  (gr_circle (center 345.28125 -5.55625) (end 350.04375 -5.55625)
+    (stroke (width 0.1) (type default)) (fill none) (layer "Edge.Cuts"))
+  (gr_circle (center 286.54375 -5.55625) (end 291.30625 -5.55625)
+    (stroke (width 0.1) (type default)) (fill none) (layer "Edge.Cuts"))
+  (gr_circle (center 110.33125 -5.55625) (end 115.09375 -5.55625)
+    (stroke (width 0.1) (type default)) (fill none) (layer "Edge.Cuts"))
+  (gr_circle (center 404.01875 -5.55625) (end 404.01875 -10.31875)
+    (stroke (width 0.1) (type default)) (fill none) (layer "Edge.Cuts"))
+  (gr_circle (center 227.80625 -5.55625) (end 232.56875 -5.55625)
+    (stroke (width 0.1) (type default)) (fill none) (layer "Edge.Cuts"))
+  (gr_circle (center -7.14375 46.0375) (end -7.14375 41.275)
+    (stroke (width 0.1) (type default)) (fill none) (layer "Edge.Cuts"))
   (group "Right hand switches" (id 6d74e477-e7b4-41d8-af0b-43ebd920e4e1)
     (members
@@
     )
   )
+  (group "" (id 32a51e92-96bf-496b-8f4b-055d9025bf5c)
+    (members
+      2843d7fa-1143-4cac-af6d-05f1cc7df869
+      3c72cff2-70a3-4ced-8e50-55594f3061ad
+      5f81c870-d999-4ba4-a59b-2d5bf3acf3ae
+      691c45fe-ba11-434f-b34f-91e5e9ec4573
+      69a7e444-1b02-4d4a-8b3e-ce57937cb248
+      69bf522e-9b55-44bf-a9cb-d1c1a0279508
+      716ef034-1bf3-4c79-91ad-d8a1e8a7e7ef
+      77240001-144c-46a9-bbe2-820cc58d769a
+      95d7085b-3343-47b2-b321-20b0b176ef7a
+      97e6a395-c0be-4e40-8d57-2666dfc23739
+      9cf6442a-d75a-4e12-83dd-88cb03fa23bb
+      a5569a8e-0edf-480c-b116-a9924d552fb1
+      af286f8c-1561-4973-9ebc-7f54f2101353
+      b84cdf78-90f7-4315-8893-4657927d43d4
+      c26f2d7d-cea0-4083-89bb-983a01797539
+      c5a7dbe6-16b4-40a5-b4fb-d9b199acc46e
+      c6e92e51-6950-42ed-88f9-f80ff149c00c
+      d4f1336d-4863-48af-a55e-839484af6d6d
+      d61e93c1-0dc5-4da2-91b1-6d0c47b51feb
+      e19f169a-1f19-4464-a909-f2fa847fc90f
+      e1f43843-04c5-47da-9c4c-59248d906b76
+      ecfdd47b-e94e-4eab-9cc1-2b481c642404
+      fb3937fa-d593-4ea5-b361-8a350b89d935
+      fd98f1d6-7166-4149-adb3-8b66b01cb3d1
+    )
+  )
